File: Launch-28020/Launch-28020_V2_routed.sch (EAGLE design)
At the start: 26 parts, among them X1 C-GRID-06-74099, X2 C-GRID-04-74099, X3 C-GRID-06-74099, X4 C-GRID-08-74099, X5 C-GRID-07-74099, X6 C-GRID-03-74099, X7 C-GRID-03-74099, X8 C-GRID-03-74099, X9 C-GRID-03-74099

Commit message: Updated Layout
Other:
- moved on the sheet: D1, J1, R4, R6, U2, X1-1, X1-2, X1-3, X1-4, X1-5, X1-6, X2-1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
